File: PowerPi.kicad_sch (KiCad schematic)
At the start: 34 parts, among them J1 2444, J3 Conn_01x02, J6 Raspberry_Pi_2_3, J8 2444, Q1 30V 4A 44mΩ, Q2 50nA 150V 200mW 200mA, Q3 30V 4A 44mΩ, U1 XL4015

Commit message: changed input capacitors to 0402 footprint and updated layout to reduce EMI
Parts:
- C2, C3: footprint Capacitor_SMD:C_0603_1608Metric -> Capacitor_SMD:C_0402_1005Metric; LCSC C15849 -> (none); ManfNum CL10A105KB8NNNC -> (none); PCBway CL10A105KB8NNNC -> (none); abv.Footprint 0603 -> 0402
Changed lines of the file:
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@@
       (effects (font (size 1.27 1.27)) (justify right))
     )
-    (property "Footprint" "Capacitor_SMD:C_0603_1608Metric" (id 2) (at 77.978 98.171 0)
+    (property "Footprint" "Capacitor_SMD:C_0402_1005Metric" (id 2) (at 77.978 98.171 0)
       (effects (font (size 1.27 1.27)) hide)
     )
@@
       (effects (font (size 1.27 1.27)) hide)
     )
-    (property "LCSC" "C15849" (id 4) (at 77.978 98.171 0)
-      (effects (font (size 1.27 1.27)) hide)
-    )
-    (property "PCBway" "CL10A105KB8NNNC" (id 5) (at 77.978 98.171 0)
-      (effects (font (size 1.27 1.27)) hide)
-    )
-    (property "abv.Footprint" "0603" (id 6) (at 77.978 98.171 0)
-      (effects (font (size 1.27 1.27)) hide)
-    )
-    (property "ManfNum" "CL10A105KB8NNNC" (id 7) (at 77.978 98.171 0)
+    (property "LCSC" "" (id 4) (at 77.978 98.171 0)
+      (effects (font (size 1.27 1.27)) hide)
+    )
+    (property "PCBway" "" (id 5) (at 77.978 98.171 0)
+      (effects (font (size 1.27 1.27)) hide)
+    )
+    (property "abv.Footprint" "0402" (id 6) (at 77.978 98.171 0)
+      (effects (font (size 1.27 1.27)) hide)
+    )
+    (property "ManfNum" "" (id 7) (at 77.978 98.171 0)
       (effects (font (size 1.27 1.27)) hide)
     )
@@
       (effects (font (size 1.27 1.27)) (justify left))
     )
-    (property "Footprint" "Capacitor_SMD:C_0603_1608Metric" (id 2) (at 67.7164 98.171 0)
+    (property "Footprint" "Capacitor_SMD:C_0402_1005Metric" (id 2) (at 67.7164 98.171 0)
       (effects (font (size 1.27 1.27)) hide)
     )
@@
       (effects (font (size 1.27 1.27)) hide)
     )
-    (property "LCSC" "C15849" (id 4) (at 67.7164 98.171 0)
-      (effects (font (size 1.27 1.27)) hide)
-    )
-    (property "PCBway" "CL10A105KB8NNNC" (id 5) (at 67.7164 98.171 0)
-      (effects (font (size 1.27 1.27)) hide)
-    )
-    (property "abv.Footprint" "0603" (id 6) (at 67.7164 98.171 0)
-      (effects (font (size 1.27 1.27)) hide)
-    )
-    (property "ManfNum" "CL10A105KB8NNNC" (id 7) (at 67.7164 98.171 0)
+    (property "LCSC" "" (id 4) (at 67.7164 98.171 0)
+      (effects (font (size 1.27 1.27)) hide)
+    )
+    (property "PCBway" "" (id 5) (at 67.7164 98.171 0)
+      (effects (font (size 1.27 1.27)) hide)
+    )
+    (property "abv.Footprint" "0402" (id 6) (at 67.7164 98.171 0)
+      (effects (font (size 1.27 1.27)) hide)
+    )
+    (property "ManfNum" "" (id 7) (at 67.7164 98.171 0)
       (effects (font (size 1.27 1.27)) hide)
     )
@@
     )
     (path "/3427c5b8-85a9-4bc0-9950-3d8f93e645b4"
-      (reference "C2") (unit 1) (value "1 uF") (footprint "Capacitor_SMD:C_0603_1608Metric")
+      (reference "C2") (unit 1) (value "1 uF") (footprint "Capacitor_SMD:C_0402_1005Metric")
     )
     (path "/227bddcb-c42b-4cd8-bc3e-9967b0269b8c"
-      (reference "C3") (unit 1) (value "1 uF") (footprint "Capacitor_SMD:C_0603_1608Metric")
+      (reference "C3") (unit 1) (value "1 uF") (footprint "Capacitor_SMD:C_0402_1005Metric")
     )
     (path "/19072074-aee5-4bd8-87b4-b7ee7fae14bf"
