File: ElectriPi.kicad_sch (KiCad schematic)
At the start: 56 parts, among them IC2 TPS51397ARJER, J1 2444, J2 JST XH 01x02, J3 JST XH 01x02, J6 Raspberry_Pi_2_3, J8 JST XH 01x02, Q1 SiA471DJ, Q2 SiA430DJT, U1 LM74700, U2 COOLING

Commit message: BOM updates
Fixed edge.cuts with fan and updated BOM
Parts:
- C1, C11, C12, C2: JLC C2179409 -> (none); LCSC (none) -> C2179409
- C10, C13, C14, C15, C17, C6, C7, C8, C9: LCSC (none) -> C2193622
- C18: JLC C2165366 -> (none); LCSC (none) -> C2165366
- C4, C5: JLC C883598 -> (none); LCSC (none) -> C312983
- D1: JLC C3712593 -> (none); LCSC (none) -> C3712593
- D4: JLC C87090 -> (none); LCSC (none) -> C87090
- D6: JLC C477955 -> (none); LCSC (none) -> C477955
- IC2: JLC C1518754 -> (none); LCSC (none) -> C1518754
- J2, J3, J8: LCSC C492456 -> C24193
- Q1: LCSC (none) -> C5918946
- Q2: JLC C727371 -> (none); LCSC (none) -> C727347
- R1, R11, R5: LCSC (none) -> C323721
- R12, R13, R3, R7: LCSC (none) -> C413107
- R14: LCSC (none) -> C319837
- R4: LCSC (none) -> C413110
- R6: LCSC C25087 -> C409028
- R8: LCSC C25867 -> C270371
- TP1, TP2, TP3, TP4, TP5, TP6: now left out of the parts list
- U1: JLC C2941042 -> (none); LCSC (none) -> C2941042
Changed lines of the file:
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@@
   )
   (symbol (lib_id "Connector:TestPoint") (at 44.45 34.29 0) (unit 1)
-    (in_bom yes) (on_board yes) (dnp no) (fields_autoplaced)
+    (in_bom no) (on_board yes) (dnp no) (fields_autoplaced)
     (property "Reference" "TP3" (at 46.228 30.9879 0)
       (effects (font (size 1.27 1.27)) (justify left))
@@
     )
     (property "Mouser" "81-GRM155R62A104KE4J" (at 102.235 43.18 0)
+      (effects (font (size 1.27 1.27)) hide)
+    )
+    (property "LCSC" "C2193622" (at 102.235 43.18 0)
       (effects (font (size 1.27 1.27)) hide)
     )
@@
       (effects (font (size 1.27 1.27)) (justify left top) hide)
     )
-    (property "JLC" "C1518754" (at 110.49 59.69 0)
+    (property "LCSC" "C1518754" (at 110.49 59.69 0)
       (effects (font (size 1.27 1.27)) hide)
     )
@@
       (effects (font (size 1.27 1.27)) hide)
     )
-    (property "JLC" "C87090" (at 67.31 54.61 90)
+    (property "LCSC" "C87090" (at 67.31 54.61 0)
       (effects (font (size 1.27 1.27)) hide)
     )
@@
     )
     (property "Mouser" "81-GRM155R62A104KE4J" (at 22.86 62.23 0)
+      (effects (font (size 1.27 1.27)) hide)
+    )
+    (property "LCSC" "C2193622" (at 22.86 62.23 0)
       (effects (font (size 1.27 1.27)) hide)
     )
@@
       (effects (font (size 1.27 1.27)) hide)
     )
-    (property "LCSC" "C492456" (at 143.51 119.38 90)
+    (property "LCSC" "C24193" (at 143.51 119.38 90)
       (effects (font (size 1.27 1.27)) hide)
     )
@@
       (effects (font (size 1.27 1.27)) hide)
     )
+    (property "LCSC" "C2193622" (at 153.67 127 0)
+      (effects (font (size 1.27 1.27)) hide)
+    )
     (pin "1")
     (pin "2")
@@
       (effects (font (size 1.27 1.27)) hide)
     )
+    (property "LCSC" "C2193622" (at 186.69 55.88 0)
+      (effects (font (size 1.27 1.27)) hide)
+    )
     (pin "1")
     (pin "2")
@@
       (effects (font (size 1.27 1.27)) hide)
     )
-    (property "JLC" "C883598" (at 196.85 55.88 0)
+    (property "LCSC" "C312983" (at 196.85 55.88 0)
       (effects (font (size 1.27 1.27)) hide)
     )
@@
       (effects (font (size 1.27 1.27)) hide)
     )
+    (property "LCSC" "C323721" (at 156.21 74.93 0)
+      (effects (font (size 1.27 1.27)) hide)
+    )
     (pin "1")
     (pin "2")
@@
       (effects (font (size 1.27 1.27)) hide)
     )
-    (property "JLC" "C2179409" (at 92.075 43.18 0)
+    (property "LCSC" "C2179409" (at 92.075 43.18 0)
       (effects (font (size 1.27 1.27)) hide)
     )
@@
       (effects (font (size 1.27 1.27)) hide)
     )
-    (property "JLC" "C2165366" (at 70.485 43.18 0)
+    (property "LCSC" "C2165366" (at 70.485 43.18 0)
       (effects (font (size 1.27 1.27)) hide)
     )
@@
       (effects (font (size 1.27 1.27)) hide)
     )
+    (property "LCSC" "C2193622" (at 49.53 119.38 0)
+      (effects (font (size 1.27 1.27)) hide)
+    )
     (pin "1")
     (pin "2")
@@
   )
   (symbol (lib_id "Connector:TestPoint") (at 27.305 111.76 0) (unit 1)
-    (in_bom yes) (on_board yes) (dnp no) (fields_autoplaced)
+    (in_bom no) (on_board yes) (dnp no) (fields_autoplaced)
     (property "Reference" "TP1" (at 29.083 108.4579 0)
       (effects (font (size 1.27 1.27)) (justify left))
@@
       (effects (font (size 1.27 1.27)) hide)
     )
+    (property "LCSC" "C2193622" (at 67.31 63.5 0)
+      (effects (font (size 1.27 1.27)) hide)
+    )
     (pin "1")
     (pin "2")
@@
       (effects (font (size 1.27 1.27)) hide)
     )
-    (property "LCSC" "C25867" (at 40.64 187.96 90)
+    (property "LCSC" "C270371" (at 40.64 187.96 90)
       (effects (font (size 1.27 1.27)) hide)
     )
@@
   )
   (symbol (lib_id "Connector:TestPoint") (at 93.98 116.84 0) (unit 1)
-    (in_bom yes) (on_board yes) (dnp no) (fields_autoplaced)
+    (in_bom no) (on_board yes) (dnp no) (fields_autoplaced)
     (property "Reference" "TP5" (at 95.758 113.5379 0)
       (effects (font (size 1.27 1.27)) (justify left))
@@
   )
   (symbol (lib_id "Connector:TestPoint") (at 39.37 88.9 0) (unit 1)
-    (in_bom yes) (on_board yes) (dnp no)
+    (in_bom no) (on_board yes) (dnp no)
     (property "Reference" "TP6" (at 41.148 85.598 0)
       (effects (font (size 1.27 1.27)) (justify left))
@@
       (effects (font (size 1.27 1.27)) hide)
     )
-    (property "LCSC" "" (at 57.15 63.5 90)
+    (property "LCSC" "C413107" (at 57.15 63.5 90)
       (effects (font (size 1.27 1.27)) hide)
     )
@@
     )
     (property "Datasheet" "~" (at 156.21 64.77 0)
+      (effects (font (size 1.27 1.27)) hide)
+    )
+    (property "LCSC" "C323721" (at 156.21 64.77 0)
       (effects (font (size 1.27 1.27)) hide)
     )
@@
       (effects (font (size 1.27 1.27)) hide)
     )
+    (property "LCSC" "C413110" (at 156.21 55.88 0)
+      (effects (font (size 1.27 1.27)) hide)
+    )
     (pin "1")
     (pin "2")
@@
     )
     (property "Datasheet" "~" (at 217.17 63.5 0)
+      (effects (font (size 1.27 1.27)) hide)
+    )
+    (property "LCSC" "C319837" (at 217.17 63.5 0)
       (effects (font (size 1.27 1.27)) hide)
     )
@@
       (effects (font (size 1.27 1.27)) hide)
     )
+    (property "LCSC" "C413107" (at 156.21 69.85 0)
+      (effects (font (size 1.27 1.27)) hide)
+    )
     (pin "1")
     (pin "2")
@@
       (effects (font (size 1.27 1.27)) hide)
     )
+    (property "LCSC" "C5918946" (at 57.15 43.18 0)
+      (effects (font (size 1.27 1.27)) hide)
+    )
     (pin "1")
     (pin "3")
@@
       (effects (font (size 1.27 1.27)) hide)
     )
-    (property "LCSC" "C25087" (at 40.64 177.8 90)
+    (property "LCSC" "C409028" (at 40.64 177.8 90)
       (effects (font (size 1.27 1.27)) hide)
     )
@@
       (effects (font (size 1.27 1.27)) hide)
     )
+    (property "LCSC" "C323721" (at 166.37 59.69 0)
+      (effects (font (size 1.27 1.27)) hide)
+    )
     (pin "1")
     (pin "2")
@@
       (effects (font (size 1.27 1.27)) hide)
     )
-    (property "JLC" "C2179409" (at 80.01 121.92 0)
+    (property "LCSC" "C2179409" (at 80.01 121.92 0)
       (effects (font (size 1.27 1.27)) hide)
     )
@@
     )
     (property "Mouser" "81-GRM155R62A104KE4J" (at 139.7 177.8 0)
+      (effects (font (size 1.27 1.27)) hide)
+    )
+    (property "LCSC" "C2193622" (at 139.7 177.8 0)
       (effects (font (size 1.27 1.27)) hide)
     )
@@
       (effects (font (size 1.27 1.27)) hide)
     )
-    (property "LCSC" "C492456" (at 31.75 78.74 0)
+    (property "LCSC" "C24193" (at 31.75 78.74 0)
       (effects (font (size 1.27 1.27)) hide)
     )
@@
     )
     (property "Datasheet" "~" (at 217.17 55.88 0)
+      (effects (font (size 1.27 1.27)) hide)
+    )
+    (property "LCSC" "C413107" (at 217.17 55.88 0)
       (effects (font (size 1.27 1.27)) hide)
     )
@@
       (effects (font (size 1.27 1.27)) hide)
     )
-    (property "JLC" "C2179409" (at 90.805 121.92 0)
+    (property "LCSC" "C2179409" (at 90.805 121.92 0)
       (effects (font (size 1.27 1.27)) hide)
     )
@@
       (effects (font (size 1.27 1.27)) hide)
     )
-    (property "JLC" "C477955" (at 22.86 127 90)
+    (property "LCSC" "C477955" (at 22.86 127 0)
       (effects (font (size 1.27 1.27)) hide)
     )
@@
       (effects (font (size 1.27 1.27)) hide)
     )
-    (property "LCSC" "C492456" (at 161.29 176.53 0)
+    (property "LCSC" "C24193" (at 161.29 176.53 0)
       (effects (font (size 1.27 1.27)) hide)
     )
@@
       (effects (font (size 1.27 1.27)) hide)
     )
+    (property "LCSC" "C2193622" (at 177.8 40.64 0)
+      (effects (font (size 1.27 1.27)) hide)
+    )
     (pin "1")
     (pin "2")
@@
       (effects (font (size 1.27 1.27)) hide)
     )
-    (property "JLC" "C883598" (at 207.01 55.88 0)
+    (property "LCSC" "C312983" (at 207.01 55.88 0)
       (effects (font (size 1.27 1.27)) hide)
     )
@@
       (effects (font (size 1.27 1.27)) hide)
     )
+    (property "LCSC" "C413107" (at 128.27 95.25 0)
+      (effects (font (size 1.27 1.27)) hide)
+    )
     (pin "1")
     (pin "2")
@@
   )
   (symbol (lib_id "Connector:TestPoint") (at 31.75 34.29 0) (unit 1)
-    (in_bom yes) (on_board yes) (dnp no) (fields_autoplaced)
+    (in_bom no) (on_board yes) (dnp no) (fields_autoplaced)
     (property "Reference" "TP2" (at 33.782 30.9879 0)
       (effects (font (size 1.27 1.27)) (justify left))
@@
   )
   (symbol (lib_id "Connector:TestPoint") (at 31.75 88.9 0) (unit 1)
-    (in_bom yes) (on_board yes) (dnp no) (fields_autoplaced)
+    (in_bom no) (on_board yes) (dnp no) (fields_autoplaced)
     (property "Reference" "TP4" (at 29.972 85.5981 0)
       (effects (font (size 1.27 1.27)) (justify right))
@@
       (effects (font (size 1.27 1.27)) hide)
     )
+    (property "LCSC" "C2193622" (at 46.99 130.81 0)
+      (effects (font (size 1.27 1.27)) hide)
+    )
     (pin "1")
     (pin "2")
@@
       (effects (font (size 1.27 1.27)) hide)
     )
-    (property "JLC" "C2179409" (at 81.915 43.18 0)
+    (property "LCSC" "C2179409" (at 81.915 43.18 0)
       (effects (font (size 1.27 1.27)) hide)
     )
@@
       (effects (font (size 1.27 1.27)) hide)
     )
-    (property "JLC" "C3712593" (at 41.91 48.26 90)
+    (property "LCSC" "C3712593" (at 41.91 48.26 0)
       (effects (font (size 1.27 1.27)) hide)
     )
@@
       (effects (font (size 1.27 1.27)) hide)
     )
-    (property "JLC" "C727371" (at 66.04 119.38 90)
+    (property "LCSC" "C727347 " (at 66.04 119.38 0)
       (effects (font (size 1.27 1.27)) hide)
     )
@@
       (effects (font (size 1.27 1.27)) hide)
     )
-    (property "JLC" "C2941042" (at 66.04 134.62 0)
-      (effects (font (size 1.27 1.27)) hide)
-    )
+    (property "LCSC" "C2941042" (at 66.04 134.62 0)
+      (effects (font (size 1.27 1.27)) hide)
+    )
